File: nixie-clock.sch (KiCad schematic (older format))
At the start: 34 parts

Commit message: finish rev a
Parts:
- removed J?: USB_B_Mini, symbol Connector:USB_B_Mini
- removed N? (x4): IN-4, nixies-us_IN-4-DSUB, symbol nixies-us:IN-4
- removed U?: nixie-step-up, symbol ronan-kicad-library:nixie-step-up
- added C10, C11, C12, C3, C9: 100nF, Capacitor_SMD:C_1206_3216Metric_Pad1.42x1.75mm_HandSolder, symbol Device:C
- added D2, D3: LED, LED_THT:LED_D5.0mm_Clear, symbol Device:LED
- added J1: Conn_01x05_Male, Connector_PinHeader_2.54mm:PinHeader_1x05_P2.54mm_Vertical, symbol Connector:Conn_01x05_Male
- added J2: Conn_01x02_Male, Connector_PinHeader_2.54mm:PinHeader_1x02_P2.54mm_Vertical, symbol Connector:Conn_01x02_Male
- added N1, N2, N3, N4: IN-4, nixies-us:IN-4-DSUB, symbol nixies-us:IN-4
- added R1, R5, R7: 10k, Resistor_SMD:R_1206_3216Metric_Pad1.42x1.75mm_HandSolder, symbol Device:R
- added R10: 110, Resistor_SMD:R_1206_3216Metric_Pad1.42x1.75mm_HandSolder, symbol Device:R
- added R13, R14: 270, Resistor_SMD:R_1206_3216Metric_Pad1.42x1.75mm_HandSolder, symbol Device:R
- added S1: 1825910-6, digikey-footprints:Switch_Tactile_THT_6x6mm, symbol dk_Tactile-Switches:1825910-6
- added U7: nixie-step-up, step-up-footprint:nixie-step-up, symbol ronan-kicad-library:nixie-step-up
- added U9: TLP627, Package_DIP:DIP-4_W7.62mm, symbol Isolator:TLP627
- C1, C2, C4, C5, C6, C7, C8: renamed from C?; footprint (none) -> Capacitor_SMD:C_1206_3216Metric_Pad1.42x1.75mm_HandSolder
- D1: renamed from D?; footprint Diode_THT:D_DO-41_SOD81_P10.16mm_Horizontal -> Diode_SMD:D_SOD-323_HandSoldering
- JP1: renamed from JP?; footprint (none) -> Jumper:SolderJumper-2_P1.3mm_Bridged_RoundedPad1.0x1.5mm
- JP2: renamed from JP?; footprint (none) -> Jumper:SolderJumper-2_P1.3mm_Open_RoundedPad1.0x1.5mm
- R11, R12, R2, R3, R4, R6, R8, R9: renamed from R?; footprint (none) -> Resistor_SMD:R_1206_3216Metric_Pad1.42x1.75mm_HandSolder
- U1, U4, U5, U8: renamed from U?; value TLP627-2 -> K155ID1; footprint Package_DIP:DIP-8_W7.62mm -> Package_DIP:DIP-16_W7.62mm
- U2, U6: renamed from U?; value TLP627-2 -> 74HC595; footprint Package_DIP:DIP-8_W7.62mm -> Package_DIP:DIP-16_W7.62mm
- U3: renamed from U?; footprint Package_DIP:DIP-8_W7.62mm -> RF_Module:ESP-12E
- gave numbers to parts that had none: 2
Connections:
- net 170V_DIGIT2_4 is gone; now on net 170V_DIGIT2-4: R3.1, R6.1, R8.1
- net VCC is gone; now on net +5V: U1.5 (VCC), U4.5 (VCC), U5.5 (VCC), U8.5 (VCC)
- net +3V3: now also C3.1, R1.1, R5.1, R7.1
- net +5V: now also C10.1, C11.1, C12.1, C9.1
- net 170V: now also U7.1 (HV), U9.4
- net GND: now also C10.2, C11.2, C12.2, C3.2, C9.2, D2.1 (K), D3.1 (K), J1.5 (Pin_5), J2.2 (Pin_2), S1.3, S1.4, U7.2 (GND), U7.3 (GND), U7.6 (GND), U9.2
- net RESET: now reaches U3.1 (REST)
- net RESET: now also J1.1 (Pin_1), R1.2, S1.1, S1.2
- net at U3.11 (GPIO2): now also R5.2
- net GPIO0: now reaches U3.12 (GPIO0)
- net GPIO0: now also J1.2 (Pin_2), R7.2
- net RXD: now reaches U3.15 (RXD)
- net RXD: now also J1.4 (Pin_4)
- net TXD: now reaches U3.16 (TXD)
- net TXD: now also J1.3 (Pin_3)
- net GPIO12: now reaches U3.6 (GPIO12)
- net GPIO12: now also R10.2
- net at U1.2 (~Q9): now also N1.0
- net at U1.16 (~Q0): now also N1.1
- net at U1.15 (~Q1): now also N1.2
- net at U1.8 (~Q2): now also N1.3
- net at U1.9 (~Q3): now also N1.4
- net at U1.13 (~Q4): now also N1.5
- net at U1.14 (~Q5): now also N1.6
- net at U1.11 (~Q6): now also N1.7
- net at U1.10 (~Q7): now also N1.8
- net at U1.1 (~Q8): now also N1.9
- net at R2.2: now also N1.A3 (A)
- net at U4.2 (~Q9): now also N2.0
- net at U4.16 (~Q0): now also N2.1
- net at U4.15 (~Q1): now also N2.2
- net at U4.8 (~Q2): now also N2.3
- net at U4.9 (~Q3): now also N2.4
- net at U4.13 (~Q4): now also N2.5
- net at U4.14 (~Q5): now also N2.6
- net at U4.11 (~Q6): now also N2.7
- net at U4.10 (~Q7): now also N2.8
- net at U4.1 (~Q8): now also N2.9
- net at R3.2: now also N2.A3 (A)
- net at U5.2 (~Q9): now also N3.0
- net at U5.16 (~Q0): now also N3.1
- net at U5.15 (~Q1): now also N3.2
- net at U5.8 (~Q2): now also N3.3
- net at U5.9 (~Q3): now also N3.4
- net at U5.13 (~Q4): now also N3.5
- net at U5.14 (~Q5): now also N3.6
- net at U5.11 (~Q6): now also N3.7
- net at U5.10 (~Q7): now also N3.8
- net at U5.1 (~Q8): now also N3.9
- net at R6.2: now also N3.A3 (A)
- net at U8.2 (~Q9): now also N4.0
- net at U8.16 (~Q0): now also N4.1
- net at U8.15 (~Q1): now also N4.2
- net at U8.8 (~Q2): now also N4.3
- net at U8.9 (~Q3): now also N4.4
- net at U8.13 (~Q4): now also N4.5
- net at U8.14 (~Q5): now also N4.6
- net at U8.11 (~Q6): now also N4.7
- net at U8.10 (~Q7): now also N4.8
- net at U8.1 (~Q8): now also N4.9
- net at R8.2: now also N4.A3 (A)
- net at D1.2 (A): now also J2.1 (Pin_1), U7.4 (5V)
- net at R9.2: now also U7.5 (EN)
- new net: R10.1, U9.1
- new net: R13.1, R14.1, U9.3
- new net: D2.2 (A), R13.2
- new net: D3.2 (A), R14.2
- no-connect marks 4 -> 10
Other:
- note added: "FLASH\n"
- note added: "INS-1 tubes\n"
